File: hardware/intervalometer-photon.sch (KiCad schematic (older format))
At the start: 6 parts, among them J3 Conn_01x02, SW1 SW_DIP_x01, U1 LTV-827, U2 Photon

Commit message: Added support for switch to start / end activity
Parts:
- J3: footprint Pin_Headers:Pin_Header_Angled_1x02_Pitch2.54mm -> Connectors_Terminal_Blocks:TerminalBlock_bornier-2_P5.08mm
Changed lines of the file:
@@
 F 0 "J3" H 7650 3100 50  0000 C CNN
 F 1 "Conn_01x02" H 7650 2800 50  0000 C CNN
-F 2 "Pin_Headers:Pin_Header_Angled_1x02_Pitch2.54mm" H 7650 3000 50  0001 C CNN
+F 2 "Connectors_Terminal_Blocks:TerminalBlock_bornier-2_P5.08mm" H 7650 3000 50  0001 C CNN
 F 3 "" H 7650 3000 50  0001 C CNN
 	1    7650 3000
